File: cc1352-swim-thermo.sch (KiCad schematic (older format))
At the start: 77 parts, among them J1 LMT_70_1, J2 LMT_70_2, J3 SMA, J4 U.FL, J5 USB_B_Micro, J6 Conn_02x05_Odd_Even, Q1 2N7002, SW1 SW_Push, U1 SKY13421-486LF, U3 CC1350F128RSM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

Commit message: Symbols done and started schema
Parts:
- removed C1, C17, C2, C3: 100nF, Capacitor_SMD:C_0603_1608Metric, symbol Device:C
- removed C10, C14, C20, C28, C29, C7: 3.6pF, Capacitor_SMD:C_0402_1005Metric, symbol Device:C
- removed C11: 100nF, Capacitor_SMD:C_0402_1005Metric, symbol Device:C
- removed C12, C19, C32: 1pF, Capacitor_SMD:C_0402_1005Metric, symbol Device:C
- removed C16: 1uF, Capacitor_SMD:C_0603_1608Metric, symbol Device:C
- removed C18, C6: 22uF, Capacitor_SMD:C_0603_1608Metric, symbol Device:C
- removed C27: DNM, Capacitor_SMD:C_0402_1005Metric, symbol Device:C
- removed C30: 5.6pF, Capacitor_SMD:C_0402_1005Metric, symbol Device:C
- removed C31: 3.3pF, Capacitor_SMD:C_0402_1005Metric, symbol Device:C
- removed C4, C5, C8, C9: 12pF, Capacitor_SMD:C_0402_1005Metric, symbol Device:C
- removed L1, L2: 10nH, Inductor_SMD:L_0402_1005Metric, symbol Device:L
- removed L11, L13, L5: 6.8nH, Inductor_SMD:L_0402_1005Metric, symbol Device:L
- removed L12: 1.5nH, Inductor_SMD:L_0402_1005Metric, symbol Device:L
- removed L14: 7.5nH, Inductor_SMD:L_0402_1005Metric, symbol Device:L
- removed L15, L4, L8: 2.2nH, Inductor_SMD:L_0402_1005Metric, symbol Device:L
- removed L3: DNM, Inductor_SMD:L_0402_1005Metric, symbol Device:L
- removed L7: 6.8uH, Inductor_SMD:L_0805_2012Metric, symbol Device:L
- removed U1: SKY13421-486LF, cc1350:SKY13421-486LF, symbol cc1350:SKY13421-486LF
- removed U3: CC1350F128RSM, cc1350:CC1350F128RSM, symbol cc1350:CC1350F128RSM
- removed Y1: 24MHz, cc1350:TSX-3225, symbol Device:Crystal_GND24
- added U?: CC1352R1F3RGZR, symbol cc1352:CC1352R1F3RGZR
- added U?: 0850BM14E0016T, symbol cc1352:0850BM14E0016T
- added U?: 2450BM14G0011T, symbol cc1350:2450BM14G0011T
- added Y?: Crystal_GND24, symbol Device:Crystal_GND24
Connections:
- net labels removed: 2_4_RF_N, 2_4_RF_P, 868_RF_N, 868_RF_P, BIAS_RF_N, BIAS_RF_P, DCDC_SW, DIO0_RF_SW_PWR, DIO1_RF_SW, VDDR
- wire segments 274 -> 134
Other:
- note removed: "2.4 GHz balun and antenna"
- note removed: "868 MHz balun and antenna"

Commit message: first schema ready
Parts:
- added C1: 1uF, symbol Device:C
- added C10, C11, C3, C5, C7, C9: 0.1uF, symbol Device:C
- added C2, C4: 12pF, symbol Device:C
- added C6, C8: 22uF, symbol Device:C
- added L1: 6.8uH, symbol Device:L
- added TP1, TP10, TP11, TP12, TP13, TP14, TP15, TP16, TP17, TP18, TP19, TP2, TP3, TP4, TP5, TP6, TP7, TP8, TP9: TestPoint, symbol Connector:TestPoint
- gave numbers to parts that had none: 4
Connections:
- net labels added: DCDC_SW, RF_N_2_4_GHZ, RF_N_SUB_1_GHZ, RF_P_2_4_GHZ, RF_P_SUB_1_GHZ, RX_TX, TAO_1, TAO_2, VDDR
- net labels removed: TAO
- wire segments 134 -> 225

Commit message: footprints and netlist
Parts:
- C1, C10, C11, C2, C3, C4, C5, C6, C7, C8, C9: footprint (none) -> Capacitor_SMD:C_0603_1608Metric
- L1: footprint (none) -> Inductor_SMD:L_0805_2012Metric
- TP1: footprint (none) -> Connector_Pin:Pin_D1.4mm_L8.5mm_W2.8mm_FlatFork
- TP10, TP11, TP12, TP13, TP14, TP15, TP16, TP17, TP18, TP19, TP2, TP3, TP4, TP5, TP6, TP7, TP8, TP9: footprint (none) -> TestPoint:TestPoint_Pad_D1.0mm
- U1: footprint (none) -> cc1352:0850BM14E0016
- U2: footprint (none) -> cc1352:CC1352R1F3RGZR
- U3: footprint (none) -> cc1350:2450BM14G011T
- Y1: footprint (none) -> cc1350:TSX-3225
Connections:
- wire segments 225 -> 226
Changed lines of the file:
@@
 F 0 "U2" H 2750 3800 50  0000 L CNN
 F 1 "CC1352R1F3RGZR" H 2450 3550 50  0000 L CNN
-F 2 "" H 3200 3100 50  0001 C CNN
+F 2 "cc1352:CC1352R1F3RGZR" H 3200 3100 50  0001 C CNN
 F 3 "" H 3200 3100 50  0001 C CNN
 	1    2800 3850
@@
 F 0 "U1" H 1175 6765 50  0000 C CNN
 F 1 "0850BM14E0016T" H 1175 6674 50  0000 C CNN
-F 2 "" V 950 6200 50  0001 C CNN
+F 2 "cc1352:0850BM14E0016" V 950 6200 50  0001 C CNN
 F 3 "" V 950 6200 50  0001 C CNN
 	1    1200 6250
@@
 F 0 "U3" V 4300 6700 60  0000 L CNN
 F 1 "2450BM14G0011T" V 3700 6350 60  0000 L CNN
-F 2 "" H 3800 6800 60  0001 C CNN
+F 2 "cc1350:2450BM14G011T" H 3800 6800 60  0001 C CNN
 F 3 "" H 3800 6800 60  0001 C CNN
 	1    4000 6800
@@
 F 0 "Y1" H 2641 1846 50  0000 L CNN
 F 1 "Crystal_GND24" H 2641 1755 50  0000 L CNN
-F 2 "" H 2450 1800 50  0001 C CNN
+F 2 "cc1350:TSX-3225" H 2450 1800 50  0001 C CNN
 F 3 "~" H 2450 1800 50  0001 C CNN
 	1    2450 1800
@@
 F 0 "C2" H 4165 1146 50  0000 L CNN
 F 1 "12pF" H 4100 1000 50  0000 L CNN
-F 2 "" H 4088 950 50  0001 C CNN
+F 2 "Capacitor_SMD:C_0603_1608Metric" H 4088 950 50  0001 C CNN
 F 3 "~" H 4050 1100 50  0001 C CNN
 	1    4050 1100
@@
 F 0 "C3" H 4465 1146 50  0000 L CNN
 F 1 "0.1uF" H 4400 1000 50  0000 L CNN
-F 2 "" H 4388 950 50  0001 C CNN
+F 2 "Capacitor_SMD:C_0603_1608Metric" H 4388 950 50  0001 C CNN
 F 3 "~" H 4350 1100 50  0001 C CNN
 	1    4350 1100
@@
 F 0 "C4" H 4765 1146 50  0000 L CNN
 F 1 "12pF" H 4700 1000 50  0000 L CNN
-F 2 "" H 4688 950 50  0001 C CNN
+F 2 "Capacitor_SMD:C_0603_1608Metric" H 4688 950 50  0001 C CNN
 F 3 "~" H 4650 1100 50  0001 C CNN
 	1    4650 1100
@@
 F 0 "C5" H 5065 1146 50  0000 L CNN
 F 1 "0.1uF" H 5000 1000 50  0000 L CNN
-F 2 "" H 4988 950 50  0001 C CNN
+F 2 "Capacitor_SMD:C_0603_1608Metric" H 4988 950 50  0001 C CNN
 F 3 "~" H 4950 1100 50  0001 C CNN
 	1    4950 1100
@@
 F 0 "C7" H 5365 1146 50  0000 L CNN
 F 1 "0.1uF" H 5300 1000 50  0000 L CNN
-F 2 "" H 5288 950 50  0001 C CNN
+F 2 "Capacitor_SMD:C_0603_1608Metric" H 5288 950 50  0001 C CNN
 F 3 "~" H 5250 1100 50  0001 C CNN
 	1    5250 1100
@@
 F 0 "C8" H 5665 1146 50  0000 L CNN
 F 1 "22uF" H 5600 1000 50  0000 L CNN
-F 2 "" H 5588 950 50  0001 C CNN
+F 2 "Capacitor_SMD:C_0603_1608Metric" H 5588 950 50  0001 C CNN
 F 3 "~" H 5550 1100 50  0001 C CNN
 	1    5550 1100
@@
 F 0 "C10" H 5965 1146 50  0000 L CNN
 F 1 "0.1uF" H 5965 1055 50  0000 L CNN
-F 2 "" H 5888 950 50  0001 C CNN
+F 2 "Capacitor_SMD:C_0603_1608Metric" H 5888 950 50  0001 C CNN
 F 3 "~" H 5850 1100 50  0001 C CNN
 	1    5850 1100
@@
 F 0 "L1" V 5040 1900 50  0000 C CNN
 F 1 "6.8uH" V 4949 1900 50  0000 C CNN
-F 2 "" H 4850 1900 50  0001 C CNN
+F 2 "Inductor_SMD:L_0805_2012Metric" H 4850 1900 50  0001 C CNN
 F 3 "~" H 4850 1900 50  0001 C CNN
 	1    4850 1900
@@
 F 0 "C6" H 5315 2096 50  0000 L CNN
 F 1 "22uF" H 5315 2005 50  0000 L CNN
-F 2 "" H 5238 1900 50  0001 C CNN
+F 2 "Capacitor_SMD:C_0603_1608Metric" H 5238 1900 50  0001 C CNN
 F 3 "~" H 5200 2050 50  0001 C CNN
 	1    5200 2050
@@
 F 0 "C9" H 5715 2096 50  0000 L CNN
 F 1 "0.1uF" H 5650 1950 50  0000 L CNN
-F 2 "" H 5638 1900 50  0001 C CNN
+F 2 "Capacitor_SMD:C_0603_1608Metric" H 5638 1900 50  0001 C CNN
 F 3 "~" H 5600 2050 50  0001 C CNN
 	1    5600 2050
@@
 F 0 "C11" H 6015 2096 50  0000 L CNN
 F 1 "0.1uF" H 5950 1950 50  0000 L CNN
-F 2 "" H 5938 1900 50  0001 C CNN
+F 2 "Capacitor_SMD:C_0603_1608Metric" H 5938 1900 50  0001 C CNN
 F 3 "~" H 5900 2050 50  0001 C CNN
 	1    5900 2050
@@
 F 0 "C1" H 3415 5346 50  0000 L CNN
 F 1 "1uF" H 3415 5255 50  0000 L CNN
-F 2 "" H 3338 5150 50  0001 C CNN
+F 2 "Capacitor_SMD:C_0603_1608Metric" H 3338 5150 50  0001 C CNN
 F 3 "~" H 3300 5300 50  0001 C CNN
 	1    3300 5300
@@
 F 0 "TP1" H 1600 4200 50  0000 R CNN
 F 1 "TestPoint" H 1492 4118 50  0001 R CNN
-F 2 "" H 1750 4000 50  0001 C CNN
+F 2 "Connector_Pin:Pin_D1.4mm_L8.5mm_W2.8mm_FlatFork" H 1750 4000 50  0001 C CNN
 F 3 "~" H 1750 4000 50  0001 C CNN
 	1    1550 4000
@@
 F 0 "TP2" H 1700 4350 50  0000 R CNN
 F 1 "TestPoint" H 1592 4268 50  0001 R CNN
-F 2 "" H 1850 4150 50  0001 C CNN
+F 2 "TestPoint:TestPoint_Pad_D1.0mm" H 1850 4150 50  0001 C CNN
 F 3 "~" H 1850 4150 50  0001 C CNN
 	1    1650 4150
@@
 F 0 "TP3" H 1800 4500 50  0000 R CNN
 F 1 "TestPoint" H 1692 4418 50  0001 R CNN
-F 2 "" H 1950 4300 50  0001 C CNN
+F 2 "TestPoint:TestPoint_Pad_D1.0mm" H 1950 4300 50  0001 C CNN
 F 3 "~" H 1950 4300 50  0001 C CNN
 	1    1750 4300
@@
 F 0 "TP4" H 1900 4650 50  0000 R CNN
 F 1 "TestPoint" H 1792 4568 50  0001 R CNN
-F 2 "" H 2050 4450 50  0001 C CNN
+F 2 "TestPoint:TestPoint_Pad_D1.0mm" H 2050 4450 50  0001 C CNN
 F 3 "~" H 2050 4450 50  0001 C CNN
 	1    1850 4450
@@
 F 0 "TP5" H 2000 4800 50  0000 R CNN
 F 1 "TestPoint" H 1892 4718 50  0001 R CNN
-F 2 "" H 2150 4600 50  0001 C CNN
+F 2 "TestPoint:TestPoint_Pad_D1.0mm" H 2150 4600 50  0001 C CNN
 F 3 "~" H 2150 4600 50  0001 C CNN
 	1    1950 4600
@@
 F 0 "TP10" V 3100 5750 50  0000 R CNN
 F 1 "TestPoint" H 3042 5568 50  0001 R CNN
-F 2 "" H 3300 5450 50  0001 C CNN
+F 2 "TestPoint:TestPoint_Pad_D1.0mm" H 3300 5450 50  0001 C CNN
 F 3 "~" H 3300 5450 50  0001 C CNN
 	1    3100 5450
@@
 F 0 "TP16" V 3850 4188 50  0000 L CNN
 F 1 "TestPoint" V 3895 4188 50  0001 L CNN
-F 2 "" H 4050 4000 50  0001 C CNN
+F 2 "TestPoint:TestPoint_Pad_D1.0mm" H 4050 4000 50  0001 C CNN
 F 3 "~" H 4050 4000 50  0001 C CNN
 	1    3850 4000
@@
 F 0 "TP19" V 4150 4288 50  0000 L CNN
 F 1 "TestPoint" V 4195 4288 50  0001 L CNN
-F 2 "" H 4350 4100 50  0001 C CNN
+F 2 "TestPoint:TestPoint_Pad_D1.0mm" H 4350 4100 50  0001 C CNN
 F 3 "~" H 4350 4100 50  0001 C CNN
 	1    4150 4100
@@
 F 0 "TP15" V 3850 3888 50  0000 L CNN
 F 1 "TestPoint" V 3895 3888 50  0001 L CNN
-F 2 "" H 4050 3700 50  0001 C CNN
+F 2 "TestPoint:TestPoint_Pad_D1.0mm" H 4050 3700 50  0001 C CNN
 F 3 "~" H 4050 3700 50  0001 C CNN
 	1    3850 3700
@@
 F 0 "TP17" V 3900 3988 50  0000 L CNN
 F 1 "TestPoint" V 3945 3988 50  0001 L CNN
-F 2 "" H 4100 3800 50  0001 C CNN
+F 2 "TestPoint:TestPoint_Pad_D1.0mm" H 4100 3800 50  0001 C CNN
 F 3 "~" H 4100 3800 50  0001 C CNN
 	1    3900 3800
@@
 F 0 "TP18" V 3950 4088 50  0000 L CNN
 F 1 "TestPoint" V 3995 4088 50  0001 L CNN
-F 2 "" H 4150 3900 50  0001 C CNN
+F 2 "TestPoint:TestPoint_Pad_D1.0mm" H 4150 3900 50  0001 C CNN
 F 3 "~" H 4150 3900 50  0001 C CNN
 	1    3950 3900
@@
 F 0 "TP14" H 3908 3374 50  0000 L CNN
 F 1 "TestPoint" H 3908 3329 50  0001 L CNN
-F 2 "" H 4050 3300 50  0001 C CNN
+F 2 "TestPoint:TestPoint_Pad_D1.0mm" H 4050 3300 50  0001 C CNN
 F 3 "~" H 4050 3300 50  0001 C CNN
 	1    3850 3300
@@
 F 0 "TP13" V 3400 2738 50  0000 L CNN
 F 1 "TestPoint" V 3445 2738 50  0001 L CNN
-F 2 "" H 3600 2550 50  0001 C CNN
+F 2 "TestPoint:TestPoint_Pad_D1.0mm" H 3600 2550 50  0001 C CNN
 F 3 "~" H 3600 2550 50  0001 C CNN
 	1    3400 2550
@@
 F 0 "TP12" V 3300 2750 50  0000 L CNN
 F 1 "TestPoint" H 3358 2579 50  0001 L CNN
-F 2 "" H 3500 2550 50  0001 C CNN
+F 2 "TestPoint:TestPoint_Pad_D1.0mm" H 3500 2550 50  0001 C CNN
 F 3 "~" H 3500 2550 50  0001 C CNN
 	1    3300 2550
@@
 F 0 "TP11" V 3200 2650 50  0000 L CNN
 F 1 "TestPoint" H 3258 2479 50  0001 L CNN
-F 2 "" H 3400 2450 50  0001 C CNN
+F 2 "TestPoint:TestPoint_Pad_D1.0mm" H 3400 2450 50  0001 C CNN
 F 3 "~" H 3400 2450 50  0001 C CNN
 	1    3200 2450
@@
 F 0 "TP9" V 3100 2550 50  0000 L CNN
 F 1 "TestPoint" H 3158 2379 50  0001 L CNN
-F 2 "" H 3300 2350 50  0001 C CNN
+F 2 "TestPoint:TestPoint_Pad_D1.0mm" H 3300 2350 50  0001 C CNN
 F 3 "~" H 3300 2350 50  0001 C CNN
 	1    3100 2350
@@
 F 0 "TP8" V 3000 2750 50  0000 L CNN
 F 1 "TestPoint" H 3058 2579 50  0001 L CNN
-F 2 "" H 3200 2550 50  0001 C CNN
+F 2 "TestPoint:TestPoint_Pad_D1.0mm" H 3200 2550 50  0001 C CNN
 F 3 "~" H 3200 2550 50  0001 C CNN
 	1    3000 2550
@@
 F 0 "TP7" V 2900 2650 50  0000 L CNN
 F 1 "TestPoint" H 2958 2479 50  0001 L CNN
-F 2 "" H 3100 2450 50  0001 C CNN
+F 2 "TestPoint:TestPoint_Pad_D1.0mm" H 3100 2450 50  0001 C CNN
 F 3 "~" H 3100 2450 50  0001 C CNN
 	1    2900 2450
@@
 F 0 "TP6" V 2800 2750 50  0000 L CNN
 F 1 "TestPoint" H 2858 2579 50  0001 L CNN
-F 2 "" H 3000 2550 50  0001 C CNN
+F 2 "TestPoint:TestPoint_Pad_D1.0mm" H 3000 2550 50  0001 C CNN
 F 3 "~" H 3000 2550 50  0001 C CNN
 	1    2800 2550
@@
 Wire Wire Line
 	4500 1900 4700 1900
+$Comp
+L power:GND #PWR0118
+U 1 1 5B7CBD44
+P 1950 3050
+F 0 "#PWR0118" H 1950 2800 50  0001 C CNN
+F 1 "GND" H 1955 2877 50  0000 C CNN
+F 2 "" H 1950 3050 50  0001 C CNN
+F 3 "" H 1950 3050 50  0001 C CNN
+	1    1950 3050
+	-1   0    0    1
+$EndComp
+Wire Wire Line
+	1950 3050 1950 3200
 $EndSCHEMATC

Commit message: started pcb
Parts:
- BT1: footprint cc1350:2_AAA_batteryholder_keystone -> Connector_Molex:Molex_KK-254_AE-6410-02A_1x02_P2.54mm_Vertical
- TP1: footprint Connector_Pin:Pin_D1.4mm_L8.5mm_W2.8mm_FlatFork -> TestPoint:TestPoint_Pad_D1.0mm
- U3: footprint cc1350:2450BM14G011T -> cc1352:0850BM14E0016
Changed lines of the file:
@@
 F 0 "BT1" H 11000 1800 50  0000 L CNN
 F 1 "Battery" H 11000 1700 50  0000 L CNN
-F 2 "cc1350:2_AAA_batteryholder_keystone" V 10900 1760 50  0001 C CNN
+F 2 "Connector_Molex:Molex_KK-254_AE-6410-02A_1x02_P2.54mm_Vertical" V 10900 1760 50  0001 C CNN
 F 3 "" V 10900 1760 50  0000 C CNN
 	1    10900 1700
@@
 F 0 "U3" V 4300 6700 60  0000 L CNN
 F 1 "2450BM14G0011T" V 3700 6350 60  0000 L CNN
-F 2 "cc1350:2450BM14G011T" H 3800 6800 60  0001 C CNN
+F 2 "cc1352:0850BM14E0016" H 3800 6800 60  0001 C CNN
 F 3 "" H 3800 6800 60  0001 C CNN
 	1    4000 6800
@@
 F 0 "TP1" H 1600 4200 50  0000 R CNN
 F 1 "TestPoint" H 1492 4118 50  0001 R CNN
-F 2 "Connector_Pin:Pin_D1.4mm_L8.5mm_W2.8mm_FlatFork" H 1750 4000 50  0001 C CNN
+F 2 "TestPoint:TestPoint_Pad_D1.0mm" H 1750 4000 50  0001 C CNN
 F 3 "~" H 1750 4000 50  0001 C CNN
 	1    1550 4000

Commit message: PCB ready for manufacturing
Parts:
- removed TP1, TP10, TP11, TP12, TP13, TP14, TP15, TP16, TP17, TP18, TP19, TP2, TP3, TP4, TP5, TP6, TP7, TP8, TP9: TestPoint, TestPoint:TestPoint_Pad_D1.0mm, symbol Connector:TestPoint
Connections:
- wire segments 226 -> 203
- no-connect marks 7 -> 27

Commit message: PCB sent to manufacturing
Parts:
- added L2: DNM, Inductor_SMD:L_0402_1005Metric, symbol Device:L
Connections:
- wire segments 203 -> 205
Changed lines of the file:
@@
 	7350 2100 7250 2100
-Wire Wire Line
-	5300 7200 5550 7200
-Wire Wire Line
-	5300 6350 5300 7200
 Wire Wire Line
 	5550 6350 5300 6350
@@
 	5850 7200 6150 7200
 Wire Wire Line
-	1150 7200 900  7200
+	1150 7200 1000 7200
 Text Notes 5450 7000 0    60   ~ 0
 Antenna matching
@@
 Wire Wire Line
 	4750 6550 4750 6650
-Wire Wire Line
-	4750 7200 5300 7200
-Connection ~ 5300 7200
 Wire Wire Line
 	4750 6950 4750 7200
@@
 NoConn ~ 3100 5100
 NoConn ~ 4750 6800
+Wire Wire Line
+	5300 6350 5300 7200
+Connection ~ 5300 7200
+Wire Wire Line
+	4750 7200 5300 7200
+Wire Wire Line
+	5300 7200 5550 7200
+$Comp
+L power:GND #PWR01
+U 1 1 5B826D08
+P 1000 7550
+F 0 "#PWR01" H 1000 7300 50  0001 C CNN
+F 1 "GND" H 1000 7400 50  0000 C CNN
+F 2 "" H 1000 7550 50  0000 C CNN
+F 3 "" H 1000 7550 50  0000 C CNN
+	1    1000 7550
+	1    0    0    -1
+$EndComp
+$Comp
+L Device:L L2
+U 1 1 5B826D0E
+P 1000 7350
+F 0 "L2" V 950 7350 50  0000 C CNN
+F 1 "DNM" V 1075 7350 50  0000 C CNN
+F 2 "Inductor_SMD:L_0402_1005Metric" H 1000 7350 50  0001 C CNN
+F 3 "" H 1000 7350 50  0000 C CNN
+	1    1000 7350
+	1    0    0    -1
+$EndComp
+Wire Wire Line
+	1000 7500 1000 7550
+Connection ~ 1000 7200
+Wire Wire Line
+	1000 7200 900  7200
 $EndSCHEMATC

Commit message: new rev of pcb
Parts:
- C10, C11, C3, C5, C7, C9: value 0.1uF -> 100nF
Changed lines of the file:
@@
 Text Label 3850 3400 0    60   ~ 0
 RESET_N
-Text Label 8850 4800 0    60   ~ 0
-VDDS
 $Comp
 L Device:R R3
@@
 Text Label 7700 950  0    60   ~ 0
 SWITCH
-Text Label 2400 5200 3    60   ~ 0
+Text Label 1850 4200 2    60   ~ 0
 SWITCH
 $Comp
@@
 Text Label 7200 3700 0    60   ~ 0
 T_ON_2
-Text Label 2700 5200 3    60   ~ 0
+Text Label 1850 4400 2    60   ~ 0
 T_ON_2
-Text Label 2600 5200 3    60   ~ 0
+Text Label 3400 2500 1    60   ~ 0
 TAO_1
-Text Label 2500 5200 3    60   ~ 0
+Text Label 1850 4300 2    60   ~ 0
 T_ON_1
 $Comp
@@
 	8150 4850 8250 4850
 Wire Wire Line
-	8850 4800 8850 4900
+	8850 4850 8850 4900
 Wire Wire Line
 	8850 5200 8850 5250
@@
 Wire Wire Line
 	10900 1000 10900 1200
-Text Label 7450 4850 2    60   ~ 0
-VDDS
-Text Label 5600 3900 2    60   ~ 0
-VDDS
-Text Label 6700 3900 2    60   ~ 0
-VDDS
 $Comp
 L power:GND #PWR058
@@
 $EndComp
 Wire Wire Line
-	7450 4850 7650 4850
-Wire Wire Line
 	7450 4950 7650 4950
 Wire Wire Line
@@
 P 4350 1100
 F 0 "C3" H 4465 1146 50  0000 L CNN
-F 1 "0.1uF" H 4400 1000 50  0000 L CNN
+F 1 "100nF" H 4400 1000 50  0000 L CNN
 F 2 "Capacitor_SMD:C_0603_1608Metric" H 4388 950 50  0001 C CNN
 F 3 "~" H 4350 1100 50  0001 C CNN
@@
 P 4950 1100
 F 0 "C5" H 5065 1146 50  0000 L CNN
-F 1 "0.1uF" H 5000 1000 50  0000 L CNN
+F 1 "100nF" H 5000 1000 50  0000 L CNN
 F 2 "Capacitor_SMD:C_0603_1608Metric" H 4988 950 50  0001 C CNN
 F 3 "~" H 4950 1100 50  0001 C CNN
@@
 P 5250 1100
 F 0 "C7" H 5365 1146 50  0000 L CNN
-F 1 "0.1uF" H 5300 1000 50  0000 L CNN
+F 1 "100nF" H 5300 1000 50  0000 L CNN
 F 2 "Capacitor_SMD:C_0603_1608Metric" H 5288 950 50  0001 C CNN
 F 3 "~" H 5250 1100 50  0001 C CNN
@@
 P 5850 1100
 F 0 "C10" H 5965 1146 50  0000 L CNN
-F 1 "0.1uF" H 5965 1055 50  0000 L CNN
+F 1 "100nF" H 5965 1055 50  0000 L CNN
 F 2 "Capacitor_SMD:C_0603_1608Metric" H 5888 950 50  0001 C CNN
 F 3 "~" H 5850 1100 50  0001 C CNN
@@
 P 5600 2050
 F 0 "C9" H 5715 2096 50  0000 L CNN
-F 1 "0.1uF" H 5650 1950 50  0000 L CNN
+F 1 "100nF" H 5650 1950 50  0000 L CNN
 F 2 "Capacitor_SMD:C_0603_1608Metric" H 5638 1900 50  0001 C CNN
 F 3 "~" H 5600 2050 50  0001 C CNN
@@
 P 5900 2050
 F 0 "C11" H 6015 2096 50  0000 L CNN
-F 1 "0.1uF" H 5950 1950 50  0000 L CNN
+F 1 "100nF" H 5950 1950 50  0000 L CNN
 F 2 "Capacitor_SMD:C_0603_1608Metric" H 5938 1900 50  0001 C CNN
 F 3 "~" H 5900 2050 50  0001 C CNN
@@
 Wire Wire Line
 	2700 2500 2700 2600
-Text Label 2800 5200 3    60   ~ 0
+Text Label 3850 3300 0    60   ~ 0
 TAO_2
 Wire Wire Line
@@
 	2300 5100 2300 5200
 Wire Wire Line
-	2400 5100 2400 5200
-Wire Wire Line
-	2500 5100 2500 5200
-Wire Wire Line
-	2600 5100 2600 5200
-Wire Wire Line
-	2700 5100 2700 5200
-Wire Wire Line
-	2800 5100 2800 5200
-Wire Wire Line
 	2900 5100 2900 5200
 Wire Wire Line
@@
 NoConn ~ 1950 4000
 NoConn ~ 1950 4100
-NoConn ~ 1950 4200
-NoConn ~ 1950 4300
-NoConn ~ 1950 4400
+NoConn ~ 2400 5100
+NoConn ~ 2500 5100
+NoConn ~ 2600 5100
 NoConn ~ 2800 2600
 NoConn ~ 2900 2600
@@
 NoConn ~ 3200 2600
 NoConn ~ 3300 2600
-NoConn ~ 3400 2600
-NoConn ~ 3750 3300
 NoConn ~ 3100 5100
 NoConn ~ 4750 6800
@@
 Wire Wire Line
 	1000 7200 900  7200
+Wire Wire Line
+	1950 4200 1850 4200
+Wire Wire Line
+	1950 4300 1850 4300
+Wire Wire Line
+	1950 4400 1850 4400
+NoConn ~ 2700 5100
+NoConn ~ 2800 5100
+Wire Wire Line
+	3400 2500 3400 2600
+Wire Wire Line
+	3850 3300 3750 3300
+$Comp
+L power:VCC #PWR0117
+U 1 1 5B9A3BD8
+P 5600 3900
+F 0 "#PWR0117" H 5600 3750 50  0001 C CNN
+F 1 "VCC" H 5617 4073 50  0000 C CNN
+F 2 "" H 5600 3900 50  0001 C CNN
+F 3 "" H 5600 3900 50  0001 C CNN
+	1    5600 3900
+	1    0    0    -1
+$EndComp
+$Comp
+L power:VCC #PWR0119
+U 1 1 5B9A3CA6
+P 6700 3900
+F 0 "#PWR0119" H 6700 3750 50  0001 C CNN
+F 1 "VCC" H 6717 4073 50  0000 C CNN
+F 2 "" H 6700 3900 50  0001 C CNN
+F 3 "" H 6700 3900 50  0001 C CNN
+	1    6700 3900
+	1    0    0    -1
+$EndComp
+$Comp
+L power:VCC #PWR0120
+U 1 1 5B9B20E3
+P 7350 4850
+F 0 "#PWR0120" H 7350 4700 50  0001 C CNN
+F 1 "VCC" H 7367 5023 50  0000 C CNN
+F 2 "" H 7350 4850 50  0001 C CNN
+F 3 "" H 7350 4850 50  0001 C CNN
+	1    7350 4850
+	1    0    0    -1
+$EndComp
+Wire Wire Line
+	7350 4850 7650 4850
+$Comp
+L power:VCC #PWR0121
+U 1 1 5B9CE581
+P 8850 4850
+F 0 "#PWR0121" H 8850 4700 50  0001 C CNN
+F 1 "VCC" H 8867 5023 50  0000 C CNN
+F 2 "" H 8850 4850 50  0001 C CNN
+F 3 "" H 8850 4850 50  0001 C CNN
+	1    8850 4850
+	1    0    0    -1
+$EndComp
 $EndSCHEMATC
